File: Kicad/macroscope/controller/controller.kicad_sch (KiCad schematic)
At the start: 0 parts

Commit message: Update Kicad files
Other:
- added sheet Mechanical (mechanical.kicad_sch)
Changed lines of the file:
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@@
     (title "Macroscope controller")
   )
-  (wire (pts (xy 88.9 73.66) (xy 107.95 73.66))
+  (wire (pts (xy 95.25 74.93) (xy 114.3 74.93))
     (stroke (width 0) (type default))
   )
-  (wire (pts (xy 88.9 76.2) (xy 107.95 76.2))
+  (wire (pts (xy 95.25 77.47) (xy 114.3 77.47))
     (stroke (width 0) (type default))
   )
-  (wire (pts (xy 88.9 63.5) (xy 107.95 63.5))
+  (wire (pts (xy 95.25 64.77) (xy 114.3 64.77))
     (stroke (width 0) (type default))
   )
-  (wire (pts (xy 88.9 50.8) (xy 107.95 50.8))
+  (wire (pts (xy 95.25 52.07) (xy 114.3 52.07))
     (stroke (width 0) (type default))
   )
-  (wire (pts (xy 88.9 48.26) (xy 107.95 48.26))
+  (wire (pts (xy 95.25 49.53) (xy 114.3 49.53))
     (stroke (width 0) (type default))
   )
-  (wire (pts (xy 88.9 78.74) (xy 107.95 78.74))
+  (wire (pts (xy 95.25 80.01) (xy 114.3 80.01))
     (stroke (width 0) (type default))
   )
-  (wire (pts (xy 88.9 60.96) (xy 107.95 60.96))
+  (wire (pts (xy 95.25 62.23) (xy 114.3 62.23))
     (stroke (width 0) (type default))
   )
-  (wire (pts (xy 88.9 66.04) (xy 107.95 66.04))
+  (wire (pts (xy 95.25 67.31) (xy 114.3 67.31))
     (stroke (width 0) (type default))
   )
-  (wire (pts (xy 88.9 53.34) (xy 107.95 53.34))
+  (wire (pts (xy 95.25 54.61) (xy 114.3 54.61))
     (stroke (width 0) (type default))
   )
-  (sheet (at 107.95 43.18) (size 21.59 40.64) (fields_autoplaced)
+  (sheet (at 114.3 44.45) (size 21.59 40.64) (fields_autoplaced)
     (stroke (width 0.1524) (type solid))
     (fill (color 0 0 0 0.0000))
-    (property "Sheetname" "Digital" (at 107.95 42.4684 0)
+    (property "Sheetname" "Digital" (at 114.3 43.7384 0)
       (effects (font (size 1.27 1.27)) (justify left bottom))
     )
-    (property "Sheetfile" "digital.kicad_sch" (at 107.95 84.4046 0)
+    (property "Sheetfile" "digital.kicad_sch" (at 114.3 85.6746 0)
       (effects (font (size 1.27 1.27)) (justify left top))
     )
-    (pin "STEPX" input (at 107.95 63.5 180)
+    (pin "STEPX" input (at 114.3 64.77 180)
       (effects (font (size 1.27 1.27)) (justify left))
     )
-    (pin "COIL1" input (at 107.95 50.8 180)
+    (pin "COIL1" input (at 114.3 52.07 180)
       (effects (font (size 1.27 1.27)) (justify left))
     )
-    (pin "COIL2" input (at 107.95 53.34 180)
+    (pin "COIL2" input (at 114.3 54.61 180)
       (effects (font (size 1.27 1.27)) (justify left))
     )
-    (pin "ENX" input (at 107.95 60.96 180)
+    (pin "ENX" input (at 114.3 62.23 180)
       (effects (font (size 1.27 1.27)) (justify left))
     )
-    (pin "DIRX" input (at 107.95 66.04 180)
+    (pin "DIRX" input (at 114.3 67.31 180)
       (effects (font (size 1.27 1.27)) (justify left))
     )
-    (pin "DIRY" input (at 107.95 78.74 180)
+    (pin "DIRY" input (at 114.3 80.01 180)
       (effects (font (size 1.27 1.27)) (justify left))
     )
-    (pin "PWM" input (at 107.95 48.26 180)
+    (pin "PWM" input (at 114.3 49.53 180)
       (effects (font (size 1.27 1.27)) (justify left))
     )
-    (pin "ENY" input (at 107.95 73.66 180)
+    (pin "ENY" input (at 114.3 74.93 180)
       (effects (font (size 1.27 1.27)) (justify left))
     )
-    (pin "STEPY" input (at 107.95 76.2 180)
+    (pin "STEPY" input (at 114.3 77.47 180)
       (effects (font (size 1.27 1.27)) (justify left))
     )
@@
     )
   )
-  (sheet (at 68.58 43.18) (size 20.32 40.64) (fields_autoplaced)
+  (sheet (at 142.24 44.45) (size 12.7 40.64) (fields_autoplaced)
     (stroke (width 0.1524) (type solid))
     (fill (color 0 0 0 0.0000))
-    (property "Sheetname" "Motion control" (at 68.58 42.4684 0)
+    (property "Sheetname" "Mechanical" (at 142.24 43.7384 0)
       (effects (font (size 1.27 1.27)) (justify left bottom))
     )
-    (property "Sheetfile" "motion_control.kicad_sch" (at 68.58 84.4046 0)
+    (property "Sheetfile" "mechanical.kicad_sch" (at 142.24 85.6746 0)
       (effects (font (size 1.27 1.27)) (justify left top))
     )
-    (pin "COIL2" input (at 88.9 53.34 0)
+    (instances
+      (project "controller"
+        (path "/87c3157d-01e1-4181-a02a-58b867324529" (page "4"))
+      )
+    )
+  )
+  (sheet (at 74.93 44.45) (size 20.32 40.64) (fields_autoplaced)
+    (stroke (width 0.1524) (type solid))
+    (fill (color 0 0 0 0.0000))
+    (property "Sheetname" "Motion control" (at 74.93 43.7384 0)
+      (effects (font (size 1.27 1.27)) (justify left bottom))
+    )
+    (property "Sheetfile" "motion_control.kicad_sch" (at 74.93 85.6746 0)
+      (effects (font (size 1.27 1.27)) (justify left top))
+    )
+    (pin "COIL2" input (at 95.25 54.61 0)
       (effects (font (size 1.27 1.27)) (justify right))
     )
-    (pin "PWM" input (at 88.9 48.26 0)
+    (pin "PWM" input (at 95.25 49.53 0)
       (effects (font (size 1.27 1.27)) (justify right))
     )
-    (pin "COIL1" input (at 88.9 50.8 0)
+    (pin "COIL1" input (at 95.25 52.07 0)
       (effects (font (size 1.27 1.27)) (justify right))
     )
-    (pin "ENX" input (at 88.9 60.96 0)
+    (pin "ENX" input (at 95.25 62.23 0)
       (effects (font (size 1.27 1.27)) (justify right))
     )
-    (pin "STEPX" input (at 88.9 63.5 0)
+    (pin "STEPX" input (at 95.25 64.77 0)
       (effects (font (size 1.27 1.27)) (justify right))
     )
-    (pin "DIRX" input (at 88.9 66.04 0)
+    (pin "DIRX" input (at 95.25 67.31 0)
       (effects (font (size 1.27 1.27)) (justify right))
     )
-    (pin "DIRY" input (at 88.9 78.74 0)
+    (pin "DIRY" input (at 95.25 80.01 0)
       (effects (font (size 1.27 1.27)) (justify right))
     )
-    (pin "STEPY" input (at 88.9 76.2 0)
+    (pin "STEPY" input (at 95.25 77.47 0)
       (effects (font (size 1.27 1.27)) (justify right))
     )
-    (pin "ENY" input (at 88.9 73.66 0)
+    (pin "ENY" input (at 95.25 74.93 0)
       (effects (font (size 1.27 1.27)) (justify right))
     )
